File: MtN1 Draft 1/MtN1 Draft 1.kicad_sch (KiCad schematic)
At the start: 47 parts, among them J1 Screw_Terminal_01x02, J10 ServoPorts_2x3, J11 QWIIC, J2 Screw_Terminal_01x02, J3 Screw_Terminal_01x02, J4 Screw_Terminal_01x02, J5 Barrel_Jack, J6 VIN, J7 GND, J9 ServoPorts_2x3, Q1 AO3401A, U1 TB6612FNG, U2 TB6612FNG, U4 MCP23017x-x-ML, U5 PCA9685BS, U7 ZSPT, U8 SY8113BADC

Commit message: Add files via upload
Parts:
- removed U7: ZSPT, Connector_PinHeader_2.54mm:PinHeader_2x03_P2.54mm_Vertical, symbol Connector_Generic:Conn_02x03_Odd_Even
- removed U8: SY8113BADC, Package_TO_SOT_SMD:SOT-23-6, symbol Connector_Generic:Conn_02x03_Odd_Even
- added C26: 10uF,25V, PCM_JLCPCB:C_0603, symbol Device:C
- added C27: 100nF, PCM_JLCPCB:C_0603, symbol Device:C
- added C28: 10pF, PCM_JLCPCB:C_0603, symbol Device:C
- added C29: 10uF, PCM_JLCPCB:C_0603, symbol Device:C
- added L3: 4.7uH, Inductor_SMD:L_1008_2520Metric, symbol Device:L
- added R10: 68kΩ, PCM_JLCPCB:R_0603, symbol Device:R
- added R12: 15kΩ, PCM_JLCPCB:R_0603, symbol Device:R
- added SW1: 5.8 ZSPT, lcsc_footprints:C2681588_SW-TH_5_8ZSPT, symbol lcsc_imported:5_8_ZSPT
- added U6, U7: SY8113BADC, lcsc_footprints:C78989_TSOT-23-6_L2_9-W1_6-P0_95-LS2_8-BR, symbol lcsc_imported:SY8113BADC
- J1, J2, J3, J4: footprint TerminalBlock_Phoenix:TerminalBlock_Phoenix_MKDS-1,5-2_1x02_P5.00mm_Horizontal -> lcsc_footprints:C8404_CONN-TH_WJ126V-5_0-2P
Connections:
- net +3V3: now also C13.2, R3.2, R6.2, U5.25 (VDD), C28.2, C29.2, L3.2, R10.1; no longer C13.1, R3.1, R6.1
- net +5V: now also C22.2, R9.1; no longer C22.1, R9.2
- net GND: now also C13.1, R11.2, C26.1, C29.1, R12.2, U6.2 (GND), U7.2 (GND); no longer C13.2, R11.1, U5.25 (VDD)
- net SCL: now also R6.1; no longer R3.2
- net SDA: now also R3.1; no longer R6.2
- net VCC: now also C26.2, U6.4 (EN), U6.5 (IN), U7.4 (EN), U7.5 (IN)
- net at C21.2: now also L2.1, U6.6 (LX)
- net at C21.1: now also U6.1 (BS); no longer L2.1
- net at J5.1: now also SW1.3
- net at Q1.3 (D): now also SW1.2
- new net: C28.1, R10.2, R12.1, U7.3 (FB)
- new net: C27.1, U7.1 (BS)
- new net: C27.2, L3.1, U7.6 (LX)
- new net: C22.1, R11.1, R9.2, U6.3 (FB)
- no-connect marks 18 -> 21
Other:
- note added: "+7.4v~8.4v"
- note added: "3V3 Buck Converter"
- note added: "5V Buck Converter"
- note added: "9v Lipo Barrel Jack"
- note added: "QWIIC Connector"
- note removed: "5v Buck Converter"
- note removed: "9v Lipo BJ"
- note removed: "QWIIC Conn"
- moved on the sheet: C10, C12, C20, C21, C22, C23, C9, D1, D2, J11, J5, J6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

Commit message: Updated project files up to Article 3
Parts:
- added J12: PQWIIC, Connector_JST:JST_SH_BM04B-SRSS-TB_1x04-1MP_P1.00mm_Vertical, symbol Connector_Generic:Conn_01x04
- added J13: GPIO_R1, symbol Connector_Generic:Conn_01x03
- added J14: GPIO_R2, symbol Connector_Generic:Conn_01x03
- added J15: GPIO_R3, symbol Connector_Generic:Conn_01x03
- added J8: GPIO_R0, symbol Connector_Generic:Conn_01x03
- added JP1: PAJP_1, symbol Jumper:SolderJumper_3_Bridged12
- added JP2: PAJP_2, symbol Jumper:SolderJumper_3_Bridged12
- added JP3: PAJP_3, symbol Jumper:SolderJumper_3_Bridged12
- added JP4: MAJP_3, symbol Jumper:SolderJumper_3_Bridged12
- added JP5: MAJP_2, symbol Jumper:SolderJumper_3_Bridged12
- added JP6: MAJP_1, symbol Jumper:SolderJumper_3_Bridged12
- added R13, R5: 10kΩ, PCM_JLCPCB:R_0603, symbol Device:R
- added R14, R15, R16, R17: 330Ω, PCM_JLCPCB:R_0603, symbol Device:R
- J1: value Screw_Terminal_01x02 -> Motor_Port_1
- J2: value Screw_Terminal_01x02 -> Motor_Port_2
- J3: value Screw_Terminal_01x02 -> Motor_Port_3
- J4: value Screw_Terminal_01x02 -> Motor_Port_4
- R1: value 10k -> 10kΩ
Connections:
- net +3V3: now also J12.2 (Pin_2), J13.2 (Pin_2), J14.2 (Pin_2), J15.2 (Pin_2), J8.2 (Pin_2), JP1.3 (B), JP2.3 (B), JP3.3 (B), JP4.3 (B), JP5.3 (B), JP6.3 (B), R13.1, R5.1; no longer U1.19 (STBY), U2.19 (STBY)
- net GND: now also J12.1 (Pin_1), J13.3 (Pin_3), J14.3 (Pin_3), J15.3 (Pin_3), J8.3 (Pin_3), JP1.1 (A), JP2.1 (A), JP3.1 (A), JP4.1 (A), JP5.1 (A), JP6.1 (A); no longer U4.11 (A0), U4.12 (A1), U4.13 (A2), U5.26 (A0), U5.27 (A1), U5.28 (A2)
- net SCL: now also J12.4 (Pin_4)
- net SDA: now also J12.3 (Pin_3)
- net at U4.25 (GPB0): now also R17.1
- net at U4.26 (GPB1): now also R16.1
- net at U4.27 (GPB2): now also R15.1
- net at U4.28 (GPB3): now also R14.1
- new net: R5.2, U1.19 (STBY)
- new net: R13.2, U2.19 (STBY)
- new net GPIO_P0: J8.1 (Pin_1), R17.2
- new net GPIO_P1: J13.1 (Pin_1), R16.2
- new net GPIO_P2: J14.1 (Pin_1), R15.2
- new net GPIO_P3: J15.1 (Pin_1), R14.2
- new net MA0: JP6.2 (C), U4.11 (A0)
- new net MA1: JP5.2 (C), U4.12 (A1)
- new net MA2: JP4.2 (C), U4.13 (A2)
- new net PA0: JP1.2 (C), U5.26 (A0)
- new net PA1: JP2.2 (C), U5.27 (A1)
- new net PA2: JP3.2 (C), U5.28 (A2)
- no-connect marks 21 -> 17
Other:
- note added: "- Motor & servo port expansion! - Qwiic expansion board! - Qwiic pass through! - Extra GPIO! - "Robust" power handling! - Simple library control!"
- note added: "- Must use a 9V lipo rechargable battery - Must be connected to any microcontroller - Microcontroller must have GND"
- note added: "- Readdressing is not for beginners! - Must use proper tools - Allowed but not recommended - GND & 3V3 tied together causes short-circuit!"
- note added: "Add. Jumpers"
- note added: "Board Capabilities"
- note added: "Board Documentation"
- note added: "Board Requirements"
- note added: "GPIO"
- note added: "MCP23017 I2C Matrix"
- note added: "Microchip I2C Address Matrices"
- note added: "NOTE!"
- note added: "PCA9685 I2C Matrix"
- note added: "QWIIC Conns."
- note removed: "QWIIC Connector"
- moved on the sheet: C1, C10, C12, C13, C14, C15, C2, C20, C21, C26, C27, C28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

Commit message: Updated project files for Article 5
Article 5 isn't done yet, but just updating files for the future when it is done.
Parts:
- C1, C12, C13, C14, C15, C2, C21, C22, C27, C28, C3, C4, C5, C6, C7, C8: footprint PCM_JLCPCB:C_0603 -> PCM_JLCPCB:C_0402
- J13, J14, J15, J8: footprint (none) -> Connector_PinSocket_2.54mm:PinSocket_1x03_P2.54mm_Vertical
- JP1, JP2, JP3, JP4, JP5, JP6: footprint (none) -> Jumper:SolderJumper-3_P1.3mm_Bridged12_RoundedPad1.0x1.5mm
- L2, L3: footprint Inductor_SMD:L_1008_2520Metric -> lcsc_footprints:C98354_IND-SMD_L2_5-W2_0_WPN252012H
- R10, R11, R12, R13, R14, R15, R16, R17, R2, R3, R4, R5, R6, R7, R8, R9: footprint PCM_JLCPCB:R_0603 -> PCM_JLCPCB:R_0402
Other:
- note added: "Default Address: 0x20"
- note added: "Default Address: 0x40"
- note removed: "Address: 0x20"
- note removed: "Address: 0x40"
Changed lines of the file:
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@@
 		)
 	)
-	(text "Address: 0x40"
+	(text "Default Address: 0x40"
 		(exclude_from_sim no)
-		(at 30.988 95.758 0)
+		(at 27.686 95.758 0)
 		(effects
 			(font
@@
 	(text "PWM Chip"
 		(exclude_from_sim no)
-		(at 31.496 92.71 0)
+		(at 24.384 92.71 0)
 		(effects
 			(font
@@
 		)
 	)
-	(text "Address: 0x20"
+	(text "Default Address: 0x20"
 		(exclude_from_sim no)
-		(at 123.444 95.25 0)
+		(at 127.254 95.25 0)
 		(effects
 			(font
@@
 			)
 		)
-		(property "Footprint" "PCM_JLCPCB:R_0603"
+		(property "Footprint" "PCM_JLCPCB:R_0402"
 			(at 65.532 113.03 90)
 			(hide yes)
@@
 			)
 		)
-		(property "Footprint" "PCM_JLCPCB:R_0603"
+		(property "Footprint" "PCM_JLCPCB:R_0402"
 			(at 79.502 176.53 90)
 			(hide yes)
@@
 			)
 		)
-		(property "Footprint" "PCM_JLCPCB:R_0603"
+		(property "Footprint" "PCM_JLCPCB:R_0402"
 			(at 144.272 71.12 90)
 			(hide yes)
@@
 			)
 		)
-		(property "Footprint" "PCM_JLCPCB:R_0603"
+		(property "Footprint" "PCM_JLCPCB:R_0402"
 			(at 73.152 113.03 90)
 			(hide yes)
@@
 			)
 		)
-		(property "Footprint" "PCM_JLCPCB:C_0603"
+		(property "Footprint" "PCM_JLCPCB:C_0402"
 			(at 48.5648 27.94 0)
 			(hide yes)
@@
 			)
 		)
-		(property "Footprint" ""
+		(property "Footprint" "Connector_PinSocket_2.54mm:PinSocket_1x03_P2.54mm_Vertical"
 			(at 161.29 132.08 0)
 			(hide yes)
@@
 			)
 		)
-		(property "Footprint" ""
+		(property "Footprint" "Jumper:SolderJumper-3_P1.3mm_Bridged12_RoundedPad1.0x1.5mm"
 			(at 160.02 53.34 0)
 			(hide yes)
@@
 			)
 		)
-		(property "Footprint" "PCM_JLCPCB:R_0603"
+		(property "Footprint" "PCM_JLCPCB:R_0402"
 			(at 210.312 43.18 90)
 			(hide yes)
@@
 			)
 		)
-		(property "Footprint" "PCM_JLCPCB:C_0603"
+		(property "Footprint" "PCM_JLCPCB:C_0402"
 			(at 66.3448 161.29 0)
 			(hide yes)
@@
 			)
 		)
-		(property "Footprint" ""
+		(property "Footprint" "Jumper:SolderJumper-3_P1.3mm_Bridged12_RoundedPad1.0x1.5mm"
 			(at 137.16 30.48 0)
 			(hide yes)
@@
 			)
 		)
-		(property "Footprint" "PCM_JLCPCB:R_0603"
+		(property "Footprint" "PCM_JLCPCB:R_0402"
 			(at 129.032 76.2 90)
 			(hide yes)
@@
 			)
 		)
-		(property "Footprint" ""
+		(property "Footprint" "Jumper:SolderJumper-3_P1.3mm_Bridged12_RoundedPad1.0x1.5mm"
 			(at 148.59 30.48 0)
 			(hide yes)
@@
 			)
 		)
-		(property "Footprint" "PCM_JLCPCB:C_0603"
+		(property "Footprint" "PCM_JLCPCB:C_0402"
 			(at 100.0252 39.37 0)
 			(hide yes)
@@
 			)
 		)
-		(property "Footprint" "PCM_JLCPCB:C_0603"
+		(property "Footprint" "PCM_JLCPCB:C_0402"
 			(at 148.8948 165.1 0)
 			(hide yes)
@@
 			)
 		)
-		(property "Footprint" "Inductor_SMD:L_1008_2520Metric"
+		(property "Footprint" "lcsc_footprints:C98354_IND-SMD_L2_5-W2_0_WPN252012H"
 			(at 72.39 161.29 0)
 			(hide yes)
@@
 			)
 		)
-		(property "Footprint" "PCM_JLCPCB:C_0603"
+		(property "Footprint" "PCM_JLCPCB:C_0402"
 			(at 204.1652 110.49 0)
 			(hide yes)
@@
 			)
 		)
-		(property "Footprint" "PCM_JLCPCB:R_0603"
+		(property "Footprint" "PCM_JLCPCB:R_0402"
 			(at 153.162 176.53 90)
 			(hide yes)
@@
 			)
 		)
-		(property "Footprint" "PCM_JLCPCB:C_0603"
+		(property "Footprint" "PCM_JLCPCB:C_0402"
 			(at 89.8652 39.37 0)
 			(hide yes)
@@
 			)
 		)
-		(property "Footprint" "PCM_JLCPCB:C_0603"
+		(property "Footprint" "PCM_JLCPCB:C_0402"
 			(at 60.6552 35.56 0)
 			(hide yes)
@@
 			)
 		)
-		(property "Footprint" "PCM_JLCPCB:R_0603"
+		(property "Footprint" "PCM_JLCPCB:R_0402"
 			(at 136.652 73.66 90)
 			(hide yes)
@@
 			)
 		)
-		(property "Footprint" ""
+		(property "Footprint" "Connector_PinSocket_2.54mm:PinSocket_1x03_P2.54mm_Vertical"
 			(at 161.29 116.84 0)
 			(hide yes)
@@
 			)
 		)
-		(property "Footprint" ""
+		(property "Footprint" "Connector_PinSocket_2.54mm:PinSocket_1x03_P2.54mm_Vertical"
 			(at 161.29 124.46 0)
 			(hide yes)
@@
 			)
 		)
-		(property "Footprint" "PCM_JLCPCB:R_0603"
+		(property "Footprint" "PCM_JLCPCB:R_0402"
 			(at 153.162 168.91 90)
 			(hide yes)
@@
 			)
 		)
-		(property "Footprint" "PCM_JLCPCB:R_0603"
+		(property "Footprint" "PCM_JLCPCB:R_0402"
 			(at 79.502 168.91 90)
 			(hide yes)
@@
 			)
 		)
-		(property "Footprint" "PCM_JLCPCB:C_0603"
+		(property "Footprint" "PCM_JLCPCB:C_0402"
 			(at 204.1652 41.91 0)
 			(hide yes)
@@
 			)
 		)
-		(property "Footprint" "PCM_JLCPCB:C_0603"
+		(property "Footprint" "PCM_JLCPCB:C_0402"
 			(at 240.9952 110.49 0)
 			(hide yes)
@@
 			)
 		)
-		(property "Footprint" "Inductor_SMD:L_1008_2520Metric"
+		(property "Footprint" "lcsc_footprints:C98354_IND-SMD_L2_5-W2_0_WPN252012H"
 			(at 146.05 161.29 0)
 			(hide yes)
@@
 			)
 		)
-		(property "Footprint" "PCM_JLCPCB:R_0603"
+		(property "Footprint" "PCM_JLCPCB:R_0402"
 			(at 100.33 188.468 90)
 			(hide yes)
@@
 			)
 		)
-		(property "Footprint" "PCM_JLCPCB:C_0603"
+		(property "Footprint" "PCM_JLCPCB:C_0402"
 			(at 194.0052 110.49 0)
 			(hide yes)
@@
 			)
 		)
-		(property "Footprint" "PCM_JLCPCB:C_0603"
+		(property "Footprint" "PCM_JLCPCB:C_0402"
 			(at 240.9952 41.91 0)
 			(hide yes)
@@
 			)
 		)
-		(property "Footprint" "PCM_JLCPCB:R_0603"
+		(property "Footprint" "PCM_JLCPCB:R_0402"
 			(at 210.312 111.76 90)
 			(hide yes)
@@
 			)
 		)
-		(property "Footprint" "PCM_JLCPCB:R_0603"
+		(property "Footprint" "PCM_JLCPCB:R_0402"
 			(at 82.042 54.61 90)
 			(hide yes)
@@
 			)
 		)
-		(property "Footprint" ""
+		(property "Footprint" "Connector_PinSocket_2.54mm:PinSocket_1x03_P2.54mm_Vertical"
 			(at 161.29 139.7 0)
 			(hide yes)
@@
 			)
 		)
-		(property "Footprint" "PCM_JLCPCB:R_0603"
+		(property "Footprint" "PCM_JLCPCB:R_0402"
 			(at 74.422 54.61 90)
 			(hide yes)
@@
 			)
 		)
-		(property "Footprint" ""
+		(property "Footprint" "Jumper:SolderJumper-3_P1.3mm_Bridged12_RoundedPad1.0x1.5mm"
 			(at 148.59 53.34 0)
 			(hide yes)
@@
 			)
 		)
-		(property "Footprint" "PCM_JLCPCB:C_0603"
+		(property "Footprint" "PCM_JLCPCB:C_0402"
 			(at 75.2348 165.1 0)
 			(hide yes)
@@
 			)
 		)
-		(property "Footprint" "PCM_JLCPCB:C_0603"
+		(property "Footprint" "PCM_JLCPCB:C_0402"
 			(at 140.0048 161.29 0)
 			(hide yes)
@@
 			)
 		)
-		(property "Footprint" "PCM_JLCPCB:R_0603"
+		(property "Footprint" "PCM_JLCPCB:R_0402"
 			(at 121.412 78.74 90)
 			(hide yes)
@@
 			)
 		)
-		(property "Footprint" ""
+		(property "Footprint" "Jumper:SolderJumper-3_P1.3mm_Bridged12_RoundedPad1.0x1.5mm"
 			(at 160.02 30.48 0)
 			(hide yes)
@@
 			)
 		)
-		(property "Footprint" "PCM_JLCPCB:R_0603"
+		(property "Footprint" "PCM_JLCPCB:R_0402"
 			(at 89.662 54.61 90)
 			(hide yes)
@@
 			)
 		)
-		(property "Footprint" "PCM_JLCPCB:C_0603"
+		(property "Footprint" "PCM_JLCPCB:C_0402"
 			(at 194.0052 41.91 0)
 			(hide yes)
@@
 			)
 		)
-		(property "Footprint" "PCM_JLCPCB:C_0603"
+		(property "Footprint" "PCM_JLCPCB:C_0402"
 			(at 251.1552 110.49 0)
 			(hide yes)
@@
 			)
 		)
-		(property "Footprint" ""
+		(property "Footprint" "Jumper:SolderJumper-3_P1.3mm_Bridged12_RoundedPad1.0x1.5mm"
 			(at 137.16 53.34 0)
 			(hide yes)
@@
 			)
 		)
-		(property "Footprint" "PCM_JLCPCB:C_0603"
+		(property "Footprint" "PCM_JLCPCB:C_0402"
 			(at 251.1552 41.91 0)
 			(hide yes)
