File: MtN1 Draft 2/MtN1 Draft 2.kicad_pcb (KiCad board)
At the start: 4 copper layers, 40 x 46 mm, 57 parts, among them J1 Motor_Port_1, J10 ServoPorts_2x3, J11 QWIIC, J12 PQWIIC, J2 Motor_Port_2, J3 Motor_Port_3, J4 Motor_Port_4, J5 Barrel_Jack, J6 VIN, J7 GND, J9 ServoPorts_2x3, Q1 AO3401A, SW1 5.8 ZSPT, U1 TB6612FNG, U2 TB6612FNG, U5 PCA9685BS, U6 SY8113BADC, U7 SY8113BADC

Commit message: Added new .STEP file
Parts:
- added G***: LOGO, LOGO, F.Cu at (126.0, 114.5)
Routing:
- net MD2 PWMB: track 10.7 -> 12.3 mm
- net GND: vias 40 -> 42
- net +3V3: vias 12 -> 13
Other:
- board text added: "5V"
- board text added: "A0"
- board text added: "A1"
- board text added: "A2"
- board text added: "Additional Help: Alfredo Systems"
- board text added: "Collaboration with: Luke Sedaca"
- board text added: "Designed By: Daniel Principe"
- board text added: "PWM"
- board text added: "v1.2"

Commit message: Draft 2 Changes; Part assignments
Parts:
- R13: footprint PCM_JLCPCB:R_0402 -> lcsc_footprints:C25744_R0402
- R9: value 36kΩ -> 33kΩ
