File: MtN1 Draft 2/MtN1 Draft 2.kicad_sch (KiCad schematic)
At the start: 55 parts, among them J1 Motor_Port_1, J10 ServoPorts_2x3, J11 QWIIC, J12 PQWIIC, J2 Motor_Port_2, J3 Motor_Port_3, J4 Motor_Port_4, J5 Barrel_Jack, J6 VIN, J7 GND, J9 ServoPorts_2x3, Q1 AO3401A, SW1 5.8 ZSPT, U1 TB6612FNG, U2 TB6612FNG, U5 PCA9685BS, U6 SY8113BADC, U7 SY8113BADC

Commit message: Draft 2 Changes; Part assignments
Parts:
- R13: footprint PCM_JLCPCB:R_0402 -> lcsc_footprints:C25744_R0402
- R9: value 36kΩ -> 33kΩ
Changed lines of the file:
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@@
 			)
 		)
-		(property "Value" "36kΩ"
+		(property "Value" "33kΩ"
 			(at 155.956 170.18 0)
 			(show_name no)
@@
 			)
 		)
-		(property "Footprint" "PCM_JLCPCB:R_0402"
+		(property "Footprint" "lcsc_footprints:C25744_R0402"
 			(at 210.312 111.76 90)
 			(hide yes)
